File: ergogen/output/pcbs/left_routed.kicad_pcb (KiCad board)
At the start: 2 copper layers, 130.6 x 90.5 mm, 59 parts

Commit message: add: v2 gerbers
Parts:
- removed DISP1: , ceoloide:display_nice_view
- added niceView1: niceView, lib:niceView_headers, F.Cu at (278.8, 153.3)
- moved H1 1.00 mm to (271.8, 171.3)
- moved RST1 0.10 mm to (286.2, 169.3)
Connections:
- D1 pad 1: P022 -> P011
- D10 pad 1: P022 -> P011
- D11 pad 1: P020 -> P100
- D12 pad 1: P017 -> P024
- D13 pad 1: P022 -> P011
- D14 pad 1: P020 -> P100
- D15 pad 1: P017 -> P024
- D16 pad 1: P022 -> P011
- D17 pad 1: P020 -> P100
- D18 pad 1: P017 -> P024
- D19 pad 1: P024 -> P104
- D2 pad 1: P020 -> P100
- D20 pad 1: P024 -> P104
- D21 pad 1: P024 -> P104
- D22 pad 1: P024 -> P104
- D23 pad 1: P017 -> P024
- D3 pad 1: P017 -> P024
- D4 pad 1: P022 -> P011
- D5 pad 1: P020 -> P100
- D6 pad 1: P017 -> P024
- D7 pad 1: P024 -> P104
- D8 pad 1: P022 -> P011
- D9 pad 1: P020 -> P100
Routing:
- net P104: track 8.37 -> 188.6 mm, vias 0 -> 2
- net P011: track 16.3 -> 192.7 mm, vias 0 -> 2
- net P100: track 0.00 -> 174.8 mm
- net P022: track 182.8 -> 17.5 mm
- net P020: track 160.3 -> 23.2 mm
- net P017: track 155.0 -> 26.8 mm
- net GND: track 100.4 -> 88.3 mm
- net RST: track 66.2 -> 55.8 mm, vias 0 -> 1
- net P024: track 177.4 -> 167.9 mm
- net VCC: track 32.2 -> 27.2 mm
- net P106: track 4.78 -> 0.00 mm
- net P029: track 135.5 -> 133.2 mm, vias 6 -> 4
- net P111: track 66.9 -> 68.4 mm, vias 6 -> 4
- net P002: track 130.2 -> 131.1 mm, vias 9 -> 7
- net P031: track 155.8 -> 155.0 mm, vias 6 -> 4
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