File: ergogen/output/pcbs/right_routed.kicad_pcb (KiCad board)
At the start: 2 copper layers, 140.9 x 96.1 mm, 88 parts

Commit message: add: generated files
Routing:
- net GND: track 0.00 -> 547.4 mm, vias 0 -> 42
- net VCC: track 0.00 -> 547.0 mm, vias 0 -> 47
- net P031: track 0.00 -> 171.7 mm, vias 0 -> 9
- net P024: track 0.00 -> 154.1 mm, vias 0 -> 10
- net P029: track 0.00 -> 151.5 mm, vias 0 -> 9
- net P002: track 0.00 -> 151.3 mm, vias 0 -> 7
- net P115: track 0.00 -> 145.3 mm, vias 0 -> 9
- net P022: track 0.00 -> 143.1 mm, vias 0 -> 10
- net P020: track 0.00 -> 128.3 mm, vias 0 -> 9
- net P017: track 0.00 -> 126.3 mm, vias 0 -> 11
- net P113: track 0.00 -> 116.3 mm, vias 0 -> 1
- net P111: track 0.00 -> 98.9 mm, vias 0 -> 4
- net LED_7: track 0.00 -> 61.8 mm, vias 0 -> 4
- net ULED_6: track 0.00 -> 61.3 mm, vias 0 -> 4
- net P010: track 0.00 -> 52.2 mm, vias 0 -> 2
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
Commit message: add: gerber files
Other:
- board text added: "Lio46 keybaord by Liolaeus"
Changed lines of the file:
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@@
 		(layer "Edge.Cuts")
+	)
+	(gr_text "Lio46 keybaord by Liolaeus"
+		(at 194.03 186.44 0)
+		(layer "B.SilkS")
+		(effects
+			(font
+				(size 1.5 1.5)
+				(thickness 0.3)
+				(bold yes)
+			)
+			(justify left bottom mirror)
+		)
 	)
 	(segment
