File: ergogen/output/pcbs/right_routed.kicad_pcb (KiCad board)
At the start: 2 copper layers, 130.6 x 90.5 mm, 59 parts

Commit message: add: v2 gerbers
Parts:
- removed DISP1: , ceoloide:display_nice_view
- added niceView1: niceView, lib:niceView_headers, F.Cu at (141.2, 153.3)
- moved H1 1.00 mm to (148.2, 171.3)
- moved RST1 0.10 mm to (133.8, 169.3)
Connections:
- D1 pad 1: P022 -> P011
- D10 pad 1: P017 -> P024
- D11 pad 1: P022 -> P011
- D12 pad 1: P020 -> P100
- D13 pad 1: P017 -> P024
- D14 pad 1: P022 -> P011
- D15 pad 1: P020 -> P100
- D16 pad 1: P017 -> P024
- D17 pad 1: P022 -> P011
- D18 pad 1: P020 -> P100
- D19 pad 1: P017 -> P024
- D2 pad 1: P020 -> P100
- D20 pad 1: P024 -> P104
- D21 pad 1: P024 -> P104
- D22 pad 1: P024 -> P104
- D23 pad 1: P024 -> P104
- D3 pad 1: P017 -> P024
- D4 pad 1: P022 -> P011
- D5 pad 1: P020 -> P100
- D6 pad 1: P017 -> P024
- D7 pad 1: P024 -> P104
- D8 pad 1: P022 -> P011
- D9 pad 1: P020 -> P100
Routing:
- net P022: track 126.0 -> 17.5 mm
- net P100: track 0.00 -> 103.7 mm
- net P011: track 16.3 -> 116.0 mm
- net P104: track 8.37 -> 106.0 mm
- net P020: track 108.6 -> 23.2 mm
- net P017: track 109.9 -> 26.8 mm
- net RST: track 67.2 -> 49.4 mm
- net P010: track 50.5 -> 58.9 mm
- net VCC: track 27.2 -> 33.1 mm, vias 1 -> 0
- net P024: track 112.6 -> 117.6 mm
- net P106: track 4.78 -> 0.00 mm
- net RAW: track 45.8 -> 41.1 mm, vias 0 -> 1
- net P002: track 153.0 -> 150.0 mm, vias 9 -> 8
- net P115: track 139.5 -> 136.7 mm, vias 9 -> 8
- net P029: track 158.6 -> 156.0 mm, vias 7 -> 6
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