File: ergogen/output/pcbs/right.kicad_pcb (KiCad board)
At the start: 2 copper layers, 130.6 x 90.5 mm, 59 parts

Commit message: add: v2 gerbers
Parts:
- moved RST1 0.10 mm to (133.8, 169.3)
Routing:
- net P031: track 177.0 -> 0.00 mm, vias 1 -> 0
- net P029: track 156.0 -> 0.00 mm, vias 6 -> 0
- net P002: track 150.0 -> 0.00 mm, vias 8 -> 0
- net P115: track 136.7 -> 0.00 mm, vias 8 -> 0
- net P024: track 117.6 -> 0.00 mm
- net P011: track 116.0 -> 0.00 mm
- net P113: track 112.7 -> 0.00 mm, vias 6 -> 0
- net P104: track 106.0 -> 0.00 mm
- net P100: track 103.7 -> 0.00 mm
- net P111: track 92.9 -> 0.00 mm, vias 6 -> 0
- net GND: track 87.3 -> 0.00 mm
- net RAW: track 44.6 -> 0.00 mm
- net P010: track 34.0 -> 0.00 mm, vias 1 -> 0
- net VCC: track 33.1 -> 0.00 mm
- net RST: track 30.3 -> 0.00 mm, vias 1 -> 0
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Other:
- net class Default added: clearance 0.2, trace_width 0.25, via_dia 0.8, via_drill 0.4
