File: ergogen/output/pcbs/right_routed2.kicad_pcb (KiCad board)
At the start: 2 copper layers, 130.6 x 90.5 mm, 59 parts

Commit message: wip: change nice view pins / reroute
Routing:
- net P010: track 34.0 -> 58.9 mm
- net RST: track 30.3 -> 48.8 mm
- net GND: track 87.3 -> 101.5 mm, vias 0 -> 1
- net RAW: track 44.6 -> 41.1 mm, vias 0 -> 1
- net mirror_pinky_bottom: track 0.00 -> 2.51 mm
- net P113: track 112.7 -> 111.0 mm
- net P111: track 92.9 -> 92.0 mm
Changed lines of the file:
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@@
+	)
+	(segment
+		(start 223.725 171.75)
+		(end 223.725 169.275)
+		(width 0.25)
+		(layer "B.Cu")
+		(net 6)
+	)
+	(segment
+		(start 223.725 169.275)
+		(end 223.7 169.25)
+		(width 0.25)
+		(layer "B.Cu")
+		(net 6)
 	)
 	(segment
@@
 	)
 	(segment
-		(start 157.1 155)
-		(end 181.225 155)
-		(width 0.25)
-		(layer "F.Cu")
-		(net 18)
-	)
-	(segment
 		(start 181.275 154.95)
 		(end 181.275 162.5)
@@
 	)
 	(segment
-		(start 181.275 148.375)
-		(end 181.275 154.95)
+		(start 156.532766 152.98)
+		(end 181.275 152.98)
 		(width 0.25)
 		(layer "F.Cu")
@@
 	)
 	(segment
-		(start 181.225 155)
-		(end 181.275 154.95)
-		(width 0.25)
-		(layer "F.Cu")
-		(net 18)
-	)
-	(segment
 		(start 134.9187 141.9887)
 		(end 149.317595 141.9887)
@@
 	)
 	(segment
+		(start 181.275 152.98)
+		(end 181.275 154.95)
+		(width 0.25)
+		(layer "F.Cu")
+		(net 18)
+	)
+	(segment
 		(start 149.317595 141.9887)
 		(end 150.5 143.171105)
@@
 	)
 	(segment
-		(start 150.5 148.4)
-		(end 157.1 155)
+		(start 150.5 143.171105)
+		(end 150.5 146.947234)
 		(width 0.25)
 		(layer "F.Cu")
@@
 	)
 	(segment
-		(start 150.5 143.171105)
-		(end 150.5 148.4)
+		(start 150.5 146.947234)
+		(end 156.532766 152.98)
+		(width 0.25)
+		(layer "F.Cu")
+		(net 18)
+	)
+	(segment
+		(start 181.275 148.375)
+		(end 181.275 152.98)
 		(width 0.25)
 		(layer "F.Cu")
@@
 	)
 	(segment
+		(start 162.581626 183.333312)
+		(end 162.581626 169.093374)
+		(width 0.25)
+		(layer "F.Cu")
+		(net 22)
+	)
+	(segment
+		(start 134.9187 144.5287)
+		(end 149.317595 144.5287)
+		(width 0.25)
+		(layer "F.Cu")
+		(net 22)
+	)
+	(segment
+		(start 163.275 157.175)
+		(end 163.275 155.725)
+		(width 0.25)
+		(layer "F.Cu")
+		(net 22)
+	)
+	(segment
+		(start 163.198314 183.95)
+		(end 162.581626 183.333312)
+		(width 0.25)
+		(layer "F.Cu")
+		(net 22)
+	)
+	(segment
+		(start 160.98 153.43)
+		(end 163.275 155.725)
+		(width 0.25)
+		(layer "F.Cu")
+		(net 22)
+	)
+	(segment
+		(start 150.05 145.261105)
+		(end 150.05 147.13363)
+		(width 0.25)
+		(layer "F.Cu")
+		(net 22)
+	)
+	(segment
+		(start 150.05 147.13363)
+		(end 156.34637 153.43)
+		(width 0.25)
+		(layer "F.Cu")
+		(net 22)
+	)
+	(segment
+		(start 162.581626 169.093374)
+		(end 163.275 168.4)
+		(width 0.25)
+		(layer "F.Cu")
+		(net 22)
+	)
+	(segment
+		(start 156.34637 153.43)
+		(end 160.98 153.43)
+		(width 0.25)
+		(layer "F.Cu")
+		(net 22)
+	)
+	(segment
 		(start 149.317595 144.5287)
 		(end 150.05 145.261105)
@@
 		(net 22)
 	)
-	(segment
-		(start 162.581626 183.333312)
-		(end 162.581626 169.093374)
-		(width 0.25)
-		(layer "F.Cu")
-		(net 22)
-	)
-	(segment
-		(start 150.05 145.261105)
-		(end 150.05 148.625)
-		(width 0.25)
-		(layer "F.Cu")
-		(net 22)
-	)
-	(segment
-		(start 150.05 148.625)
-		(end 157.15 155.725)
-		(width 0.25)
-		(layer "F.Cu")
-		(net 22)
-	)
-	(segment
-		(start 163.275 157.175)
-		(end 163.275 155.725)
-		(width 0.25)
-		(layer "F.Cu")
-		(net 22)
-	)
-	(segment
-		(start 163.198314 183.95)
-		(end 162.581626 183.333312)
-		(width 0.25)
-		(layer "F.Cu")
-		(net 22)
-	)
-	(segment
-		(start 157.15 155.725)
-		(end 163.275 155.725)
-		(width 0.25)
-		(layer "F.Cu")
-		(net 22)
-	)
-	(segment
-		(start 134.9187 144.5287)
-		(end 149.317595 144.5287)
-		(width 0.25)
-		(layer "F.Cu")
-		(net 22)
-	)
-	(segment
-		(start 162.581626 169.093374)
-		(end 163.275 168.4)
-		(width 0.25)
-		(layer "F.Cu")
-		(net 22)
-	)
 	(via
 		(at 163.275 168.4)
@@
 	)
 	(segment
+		(start 142.375 148.165)
+		(end 139.94 145.73)
+		(width 0.25)
+		(layer "B.Cu")
+		(net 29)
+	)
+	(segment
 		(start 136.343206 184.341209)
 		(end 136.343206 179.30342)
@@
 	)
 	(segment
+		(start 136.343206 179.30342)
+		(end 142.375 173.271626)
+		(width 0.25)
+		(layer "B.Cu")
+		(net 29)
+	)
+	(segment
 		(start 137.061322 194.150231)
 		(end 137.061322 185.059325)
@@
 	)
 	(segment
-		(start 136.343206 179.30342)
-		(end 144.94 170.706626)
+		(start 142.375 173.271626)
+		(end 142.375 148.165)
 		(width 0.25)
 		(layer "B.Cu")
@@
 	)
 	(segment
-		(start 142.565 152.82)
-		(end 142.565 148.095)
+		(start 135.335 160.05)
+		(end 135.335 159.005)
 		(width 0.25)
 		(layer "F.Cu")
@@
 	)
 	(segment
-		(start 135.335 160.05)
-		(end 142.565 152.82)
+		(start 135.335 159.005)
+		(end 135.33 159)
 		(width 0.25)
 		(layer "F.Cu")
 		(net 35)
 	)
-	(segment
-		(start 142.565 148.095)
-		(end 142.56 148.09)
-		(width 0.25)
-		(layer "F.Cu")
+	(via
+		(at 135.33 159)
+		(size 0.8)
+		(drill 0.4)
+		(layers "F.Cu" "B.Cu")
 		(net 35)
 	)
@@
 	)
 	(segment
+		(start 134.4 158.07)
+		(end 135.33 159)
+		(width 0.25)
+		(layer "B.Cu")
+		(net 35)
+	)
+	(segment
+		(start 134.4 150.0826)
+		(end 134.4 158.07)
+		(width 0.25)
+		(layer "B.Cu")
+		(net 35)
+	)
+	(segment
+		(start 135.2313 149.2513)
+		(end 134.4 150.0826)
+		(width 0.25)
+		(layer "B.Cu")
+		(net 35)
+	)
+	(segment
 		(start 135.2313 121.9813)
 		(end 135.2313 149.2513)
@@
 	)
 	(segment
+		(start 135.024694 153.625)
+		(end 142.115 153.625)
+		(width 0.25)
+		(layer "F.Cu")
+		(net 36)
+	)
+	(segment
 		(start 132.85 171.925)
 		(end 132.85 172.2)
@@
 	)
 	(segment
+		(start 142.115 153.625)
+		(end 143.74 152)
+		(width 0.25)
+		(layer "F.Cu")
+		(net 36)
+	)
+	(segment
+		(start 132.594847 151.195153)
+		(end 135.024694 153.625)
+		(width 0.25)
+		(layer "F.Cu")
+		(net 36)
+	)
+	(via
+		(at 132.594847 151.195153)
+		(size 0.8)
+		(drill 0.4)
+		(layers "F.Cu" "B.Cu")
+		(net 36)
+	)
+	(segment
+		(start 132.3787 150.979006)
+		(end 132.3787 124.0713)
+		(width 0.25)
+		(layer "B.Cu")
+		(net 36)
+	)
+	(segment
 		(start 132.3787 124.0713)
-		(end 132.3787 149.9537)
+		(end 133.58 122.87)
 		(width 0.25)
 		(layer "B.Cu")
@@
 	)
 	(segment
-		(start 133.58 122.87)
-		(end 132.3787 124.0713)
+		(start 132.594847 151.195153)
+		(end 132.3787 150.979006)
 		(width 0.25)
 		(layer "B.Cu")
@@
 	(segment
 		(start 134.55 166.675)
-		(end 134.55 165.33)
+		(end 134.55 165.85)
 		(width 0.25)
 		(layer "F.Cu")
@@
 		(net 37)
 	)
-	(via
-		(at 134.55 165.33)
-		(size 0.8)
-		(drill 0.4)
-		(layers "F.Cu" "B.Cu")
+	(segment
+		(start 134.55 165.85)
+		(end 133.72 165.02)
+		(width 0.25)
+		(layer "F.Cu")
+		(net 37)
+	)
+	(via
+		(at 133.72 165.02)
+		(size 0.8)
+		(drill 0.4)
+		(layers "F.Cu" "B.Cu")
+		(net 37)
+	)
+	(segment
+		(start 134.7813 126.6113)
+		(end 134.7813 149.0587)
+		(width 0.25)
+		(layer "B.Cu")
+		(net 37)
+	)
+	(segment
+		(start 132.75 156.51)
+		(end 132.75 164.05)
+		(width 0.25)
+		(layer "B.Cu")
+		(net 37)
+	)
+	(segment
+		(start 133.95 155.31)
+		(end 132.75 156.51)
+		(width 0.25)
+		(layer "B.Cu")
 		(net 37)
 	)
@@
 	)
 	(segment
-		(start 134.7813 126.6113)
-		(end 134.7813 148.43)
-		(width 0.25)
-		(layer "B.Cu")
+		(start 133.95 149.89)
+		(end 133.95 155.31)
+		(width 0.25)
+		(layer "B.Cu")
+		(net 37)
+	)
+	(segment
+		(start 134.7813 149.0587)
+		(end 133.95 149.89)
+		(width 0.25)
+		(layer "B.Cu")
+		(net 37)
+	)
+	(segment
+		(start 132.75 164.05)
+		(end 133.72 165.02)
+		(width 0.25)
+		(layer "B.Cu")
